Commit message: feat: add LDJY retargeting tools and OpenArm simulation

File: ldjy_retargeting/assets/robots/ldjy_hand/urdf/ldjy_left_hand.urdf (robot description, URDF)
Before this commit: robot ldjy_left_hand, 27 links, 26 joints
Joints:
- joint left_finger1_tip_fixed: origin xyz=5.12946368656e-18 -0.000898255926846 0.029586045233 rpy=0 0 0 -> xyz=3.94010968055e-18 -0.000594787785201 0.0195906509393 rpy=0 0 0
- joint left_finger2_tip_fixed: origin xyz=-3.22520490779e-19 -0.000825056643836 0.0295881765594 rpy=0 0 0 -> xyz=-3.39113037287e-19 -0.000546318254652 0.0195920620687 rpy=0 0 0
- joint left_finger3_tip_fixed: origin xyz=1.45513261078e-12 0.000427597164136 0.0295965928695 rpy=0 0 0 -> xyz=9.63529011583e-13 0.000283137108652 0.0195976363593 rpy=0 0 0
- joint left_finger4_tip_fixed: origin xyz=0.000202119138782 -0.00184365112833 0.0398611378018 rpy=0 0 0 -> xyz=0.000151468124729 -0.00138163253983 0.0298719449766 rpy=0 0 0
- joint left_thumb_tip_fixed: origin xyz=-3.00852510204e-18 -0.0399322083726 0.00321148415111 rpy=0 0 0 -> xyz=-2.39495233588e-18 -0.0303631046125 0.00244190424761 rpy=0 0 0

File: ldjy_retargeting/assets/robots/ldjy_hand/urdf/ldjy_right_hand.urdf (robot description, URDF)
Before this commit: robot ldjy_right_hand, 27 links, 26 joints
Joints:
- joint right_finger1_tip_fixed: origin xyz=-5.12946368656e-18 -0.000898255926846 0.029586045233 rpy=0 0 0 -> xyz=-3.94010968055e-18 -0.000594787785201 0.0195906509393 rpy=0 0 0
- joint right_finger2_tip_fixed: origin xyz=3.22520490779e-19 -0.000825056643836 0.0295881765594 rpy=0 0 0 -> xyz=3.39113037287e-19 -0.000546318254652 0.0195920620687 rpy=0 0 0
- joint right_finger3_tip_fixed: origin xyz=-1.45513261078e-12 0.000427597164136 0.0295965928695 rpy=0 0 0 -> xyz=-9.63529011583e-13 0.000283137108652 0.0195976363593 rpy=0 0 0
- joint right_finger4_tip_fixed: origin xyz=-0.000202119138782 -0.00184365112833 0.0398611378018 rpy=0 0 0 -> xyz=-0.000151468124729 -0.00138163253983 0.0298719449766 rpy=0 0 0
- joint right_thumb_tip_fixed: origin xyz=3.00852510204e-18 -0.0399322083726 0.00321148415111 rpy=0 0 0 -> xyz=2.39495233588e-18 -0.0303631046125 0.00244190424761 rpy=0 0 0

Commit message: feat: add LDJY tuning workflows and WiLoR input

File: ldjy_retargeting/assets/robots/ldjy_hand/urdf/ldjy_left_hand.urdf (robot description, URDF)
Before this commit: robot ldjy_left_hand, 27 links, 26 joints
Links:
- added link left_finger1_pad_frame
- added link left_finger2_pad_frame
- added link left_finger3_pad_frame
- added link left_finger4_pad_frame
- added link left_thumb_pad_frame
Joints:
- added joint left_finger1_pad_frame_fixed: type fixed, parent left_finger1_link4, child left_finger1_pad_frame, origin xyz=0.000650000000021 0.00450561490379 0.0203260926594 rpy=4.01167987718e-12 1.54044485282 1.57079632679
- added joint left_finger2_pad_frame_fixed: type fixed, parent left_finger2_link4, child left_finger2_pad_frame, origin xyz=0.000650000000024 0.0045558878015 0.0203148834496 rpy=4.7474246756e-12 1.54291887718 1.57079632679
- added joint left_finger3_pad_frame_fixed: type fixed, parent left_finger3_link4, child left_finger3_pad_frame, origin xyz=0.000650000001009 0.00541135856617 0.0201039253082 rpy=3.14159265019 1.55634981875 -1.5707963302
- added joint left_finger4_pad_frame_fixed: type fixed, parent left_finger4_link4, child left_finger4_pad_frame, origin xyz=-0.000527520904337 0.00552645560218 0.0306411188614 rpy=0.127174305269 1.52430090344 1.67999008312
- added joint left_thumb_pad_frame_fixed: type fixed, parent left_thumb_link4, child left_thumb_pad_frame, origin xyz=0.00057 -0.030054383314 0.0124619777339 rpy=0 0.0802506835855 1.57079632679
- joint left_finger1_tip_fixed: origin xyz=3.94010968055e-18 -0.000594787785201 0.0195906509393 rpy=0 0 0 -> xyz=1.72390144159e-14 0.00339976361945 0.0297165365339 rpy=0 0 0
- joint left_finger2_tip_fixed: origin xyz=-3.39113037287e-19 -0.000546318254652 0.0195920620687 rpy=0 0 0 -> xyz=2.09409077649e-14 0.00357323373205 0.0297108214506 rpy=0 0 0
- joint left_finger3_tip_fixed: origin xyz=9.63529011583e-13 0.000283137108652 0.0195976363593 rpy=0 0 0 -> xyz=1.4761443315e-12 0.00682692933065 0.029504138434 rpy=0 0 0
- joint left_finger4_tip_fixed: origin xyz=0.000151468124729 -0.00138163253983 0.0298719449766 rpy=0 0 0 -> xyz=0.000305268631489 0.00384935354031 0.0401239267378 rpy=0 0 0
- joint left_thumb_tip_fixed: origin xyz=-2.39495233588e-18 -0.0303631046125 0.00244190424761 rpy=0 0 0 -> xyz=-3.00852510204e-18 -0.0399322083726 0.00321148415111 rpy=0 0 0

File: ldjy_retargeting/assets/robots/ldjy_hand/urdf/ldjy_right_hand.urdf (robot description, URDF)
Before this commit: robot ldjy_right_hand, 27 links, 26 joints
Links:
- added link right_finger1_pad_frame
- added link right_finger2_pad_frame
- added link right_finger3_pad_frame
- added link right_finger4_pad_frame
- added link right_thumb_pad_frame
Joints:
- added joint right_finger1_pad_frame_fixed: type fixed, parent right_finger1_link4, child right_finger1_pad_frame, origin xyz=-0.000650000000021 0.00450561490379 0.0203260926594 rpy=4.01212396639e-12 -1.54044485282 -1.57079632679
- added joint right_finger2_pad_frame_fixed: type fixed, parent right_finger2_link4, child right_finger2_pad_frame, origin xyz=-0.000650000000024 0.0045558878015 0.0203148834496 rpy=4.75341987993e-12 -1.54291887718 -1.57079632679
- added joint right_finger3_pad_frame_fixed: type fixed, parent right_finger3_link4, child right_finger3_pad_frame, origin xyz=-0.000650000001009 0.00541135856617 0.0201039253082 rpy=3.14159265019 -1.55634981875 1.5707963302
- added joint right_finger4_pad_frame_fixed: type fixed, parent right_finger4_link4, child right_finger4_pad_frame, origin xyz=0.000527520904337 0.00552645560218 0.0306411188614 rpy=0.127174305269 -1.52430090344 -1.67999008312
- added joint right_thumb_pad_frame_fixed: type fixed, parent right_thumb_link4, child right_thumb_pad_frame, origin xyz=-0.00057 -0.030054383314 0.0124619777339 rpy=0 -0.0802506835855 -1.57079632679
- joint right_finger1_tip_fixed: origin xyz=-3.94010968055e-18 -0.000594787785201 0.0195906509393 rpy=0 0 0 -> xyz=-1.72390144159e-14 0.00339976361945 0.0297165365339 rpy=0 0 0
- joint right_finger2_tip_fixed: origin xyz=3.39113037287e-19 -0.000546318254652 0.0195920620687 rpy=0 0 0 -> xyz=-2.09409077649e-14 0.00357323373205 0.0297108214506 rpy=0 0 0
- joint right_finger3_tip_fixed: origin xyz=-9.63529011583e-13 0.000283137108652 0.0195976363593 rpy=0 0 0 -> xyz=-1.4761443315e-12 0.00682692933065 0.029504138434 rpy=0 0 0
- joint right_finger4_tip_fixed: origin xyz=-0.000151468124729 -0.00138163253983 0.0298719449766 rpy=0 0 0 -> xyz=-0.000305268631489 0.00384935354031 0.0401239267378 rpy=0 0 0
- joint right_thumb_tip_fixed: origin xyz=2.39495233588e-18 -0.0303631046125 0.00244190424761 rpy=0 0 0 -> xyz=3.00852510204e-18 -0.0399322083726 0.00321148415111 rpy=0 0 0

File: ldjy_retargeting/assets/robots/openarm_hand/urdf/openarm_bimanual_mano.urdf (robot description, URDF)
Before this commit: robot openarm_bimanual_mano, 72 links, 71 joints
Links:
- added link left_finger1_pad_frame
- added link left_finger2_pad_frame
- added link left_finger3_pad_frame
- added link left_finger4_pad_frame
- added link left_thumb_pad_frame
- added link right_finger1_pad_frame
- added link right_finger2_pad_frame
- added link right_finger3_pad_frame
- added link right_finger4_pad_frame
- added link right_thumb_pad_frame
Joints:
- added joint left_finger1_pad_frame_fixed: type fixed, parent left_finger1_link4, child left_finger1_pad_frame, origin xyz=0.000649999999962 0.00450561490399 0.0203260926594 rpy=3.9944714203e-12 1.54044485282 1.57079632679
- added joint left_finger2_pad_frame_fixed: type fixed, parent left_finger2_link4, child left_finger2_pad_frame, origin xyz=0.000649999999966 0.00455588780148 0.0203148834496 rpy=4.74242867199e-12 1.54291887718 1.57079632679
- added joint left_finger3_pad_frame_fixed: type fixed, parent left_finger3_link4, child left_finger3_pad_frame, origin xyz=0.000650000000969 0.00541135856597 0.0201039253082 rpy=3.14159265019 1.55634981875 -1.5707963302
- added joint left_finger4_pad_frame_fixed: type fixed, parent left_finger4_link4, child left_finger4_pad_frame, origin xyz=-0.000527520904384 0.00552645560178 0.0306411188614 rpy=0.127174305263 1.52430090344 1.67999008311
- added joint left_thumb_pad_frame_fixed: type fixed, parent left_thumb_link4, child left_thumb_pad_frame, origin xyz=0.000569999999648 -0.0300543833141 0.0124619777338 rpy=3.94084764821e-12 0.0802506835854 1.57079632679
- added joint right_finger1_pad_frame_fixed: type fixed, parent right_finger1_link4, child right_finger1_pad_frame, origin xyz=-0.00065000000008 0.00450561490359 0.0203260926594 rpy=4.00890431962e-12 -1.54044485282 -1.57079632679
- added joint right_finger2_pad_frame_fixed: type fixed, parent right_finger2_link4, child right_finger2_pad_frame, origin xyz=-0.000650000000082 0.00455588780152 0.0203148834496 rpy=4.76330086485e-12 -1.54291887718 -1.57079632679
- added joint right_finger3_pad_frame_fixed: type fixed, parent right_finger3_link4, child right_finger3_pad_frame, origin xyz=-0.000650000001049 0.00541135856637 0.0201039253082 rpy=3.14159265019 -1.55634981875 1.5707963302
- added joint right_finger4_pad_frame_fixed: type fixed, parent right_finger4_link4, child right_finger4_pad_frame, origin xyz=0.00052752090429 0.00552645560258 0.0306411188614 rpy=0.127174305275 -1.52430090344 -1.67999008313
- added joint right_thumb_pad_frame_fixed: type fixed, parent right_thumb_link4, child right_thumb_pad_frame, origin xyz=-0.000570000000351 -0.0300543833139 0.012461977734 rpy=-3.94118071512e-12 -0.0802506835856 -1.57079632679
- joint left_finger1_tip_fixed: origin xyz=-8.313089031e-14 -0.000594787784997 0.0195906509393 rpy=0 0 0 -> xyz=-4.66040959013e-14 0.00339976361966 0.0297165365339 rpy=0 0 0
- joint left_finger2_tip_fixed: origin xyz=-8.32577350079e-14 -0.000546318254664 0.0195920620687 rpy=0 0 0 -> xyz=-4.21546260539e-14 0.00357323373204 0.0297108214506 rpy=0 0 0
- joint left_finger3_tip_fixed: origin xyz=8.98705259942e-13 0.000283137108452 0.0195976363593 rpy=0 0 0 -> xyz=1.44288901641e-12 0.00682692933044 0.029504138434 rpy=0 0 0
- joint left_finger4_tip_fixed: origin xyz=0.000151468124651 -0.00138163254023 0.0298719449766 rpy=0 0 0 -> xyz=0.000305268631434 0.00384935353989 0.0401239267378 rpy=0 0 0
- joint left_thumb_tip_fixed: origin xyz=-3.91759923302e-13 -0.0303631046126 0.00244190424752 rpy=0 0 0 -> xyz=-4.16695657022e-13 -0.0399322083727 0.00321148415102 rpy=0 0 0
- joint right_finger1_tip_fixed: origin xyz=-8.31240070306e-14 -0.000594787785405 0.0195906509393 rpy=0 0 0 -> xyz=-8.1072751647e-14 0.00339976361924 0.0297165365339 rpy=0 0 0
- joint right_finger2_tip_fixed: origin xyz=-8.32625555493e-14 -0.00054631825464 0.0195920620687 rpy=0 0 0 -> xyz=-8.40410678071e-14 0.00357323373206 0.0297108214506 rpy=0 0 0
- joint right_finger3_tip_fixed: origin xyz=-1.02832168657e-12 0.000283137108852 0.0195976363593 rpy=0 0 0 -> xyz=-1.50935104949e-12 0.00682692933086 0.029504138434 rpy=0 0 0
- joint right_finger4_tip_fixed: origin xyz=-0.000151468124807 -0.00138163253943 0.0298719449766 rpy=0 0 0 -> xyz=-0.000305268631544 0.00384935354073 0.0401239267378 rpy=0 0 0
- joint right_thumb_tip_fixed: origin xyz=-3.9175984588e-13 -0.0303631046124 0.0024419042477 rpy=0 0 0 -> xyz=-4.16686502887e-13 -0.0399322083725 0.0032114841512 rpy=0 0 0

Commit message: feat: add MANO-LDJY pad calibration and registration

File: ldjy_retargeting/assets/robots/ldjy_hand/urdf/ldjy_left_hand.urdf (robot description, URDF)
Before this commit: robot ldjy_left_hand, 32 links, 31 joints
Links:
- removed link left_finger1_pad_frame
- removed link left_finger2_pad_frame
- removed link left_finger3_pad_frame
- removed link left_finger4_pad_frame
- removed link left_thumb_pad_frame
- added link left_finger1_pad
- added link left_finger2_pad
- added link left_finger3_pad
- added link left_finger4_pad
- added link left_thumb_pad
Joints:
- removed joint left_finger1_pad_frame_fixed
- removed joint left_finger2_pad_frame_fixed
- removed joint left_finger3_pad_frame_fixed
- removed joint left_finger4_pad_frame_fixed
- removed joint left_thumb_pad_frame_fixed
- added joint left_finger1_pad_fixed: type fixed, parent left_finger1_link4, child left_finger1_pad, origin xyz=0.000887896997077 -0.00739003330634 0.0202260113406 rpy=0 0 0
- added joint left_finger2_pad_fixed: type fixed, parent left_finger2_link4, child left_finger2_pad, origin xyz=0.000345141712275 -0.00717387617459 0.0207279644612 rpy=0 0 0
- added joint left_finger3_pad_fixed: type fixed, parent left_finger3_link4, child left_finger3_pad, origin xyz=0.000646578946653 -0.00638898613424 0.0207611224125 rpy=0 0 0
- added joint left_finger4_pad_fixed: type fixed, parent left_finger4_link4, child left_finger4_pad, origin xyz=-0.000717825545034 -0.00652127833713 0.030480346822 rpy=0 0 0
- added joint left_thumb_pad_fixed: type fixed, parent left_thumb_link4, child left_thumb_pad, origin xyz=3.66216494593e-05 -0.028500341515 0.0127727528254 rpy=0 0 0

File: ldjy_retargeting/assets/robots/ldjy_hand/urdf/ldjy_right_hand.urdf (robot description, URDF)
Before this commit: robot ldjy_right_hand, 32 links, 31 joints
Links:
- removed link right_finger1_pad_frame
- removed link right_finger2_pad_frame
- removed link right_finger3_pad_frame
- removed link right_finger4_pad_frame
- removed link right_thumb_pad_frame
- added link right_finger1_pad
- added link right_finger2_pad
- added link right_finger3_pad
- added link right_finger4_pad
- added link right_thumb_pad
Joints:
- removed joint right_finger1_pad_frame_fixed
- removed joint right_finger2_pad_frame_fixed
- removed joint right_finger3_pad_frame_fixed
- removed joint right_finger4_pad_frame_fixed
- removed joint right_thumb_pad_frame_fixed
- added joint right_finger1_pad_fixed: type fixed, parent right_finger1_link4, child right_finger1_pad, origin xyz=-0.000887896997077 -0.00739003330634 0.0202260113406 rpy=0 0 0
- added joint right_finger2_pad_fixed: type fixed, parent right_finger2_link4, child right_finger2_pad, origin xyz=-0.000345141712275 -0.00717387617459 0.0207279644612 rpy=0 0 0
- added joint right_finger3_pad_fixed: type fixed, parent right_finger3_link4, child right_finger3_pad, origin xyz=-0.000646578946653 -0.00638898613424 0.0207611224125 rpy=0 0 0
- added joint right_finger4_pad_fixed: type fixed, parent right_finger4_link4, child right_finger4_pad, origin xyz=0.000717825545034 -0.00652127833713 0.030480346822 rpy=0 0 0
- added joint right_thumb_pad_fixed: type fixed, parent right_thumb_link4, child right_thumb_pad, origin xyz=-3.66216494593e-05 -0.028500341515 0.0127727528254 rpy=0 0 0

Commit message: feat: add MANO pad pose retargeting

File: ldjy_retargeting/assets/robots/ldjy_hand/urdf/ldjy_left_hand.urdf (robot description, URDF)
Before this commit: robot ldjy_left_hand, 32 links, 31 joints
Joints:
- joint left_finger1_pad_fixed: origin xyz=0.000887896997077 -0.00739003330634 0.0202260113406 rpy=0 0 0 -> xyz=0.000887896997077 -0.00739003330634 0.0202260113406 rpy=1.24252620701 7.13747252412e-08 5.10912838703e-08
- joint left_finger2_pad_fixed: origin xyz=0.000345141712275 -0.00717387617459 0.0207279644612 rpy=0 0 0 -> xyz=0.000345141712275 -0.00717387617459 0.0207279644612 rpy=1.24005577254 -1.45069127377e-07 -1.03572263987e-07
- joint left_finger3_pad_fixed: origin xyz=0.000646578946653 -0.00638898613424 0.0207611224125 rpy=0 0 0 -> xyz=0.000646578946653 -0.00638898613424 0.0207611224125 rpy=1.19772648334 -1.19549859345e-07 -8.15891079142e-08
- joint left_finger4_pad_fixed: origin xyz=-0.000717825545034 -0.00652127833713 0.030480346822 rpy=0 0 0 -> xyz=-0.000717825545034 -0.00652127833713 0.030480346822 rpy=1.19832174357 -9.54065941805e-08 -6.51537008789e-08
- joint left_retarget_wrist_fixed: origin xyz=-0.015 -0 0.03 rpy=0 0 1.57079632679 -> xyz=-0.0145034869034 -0.0111925861623 0.0251133508706 rpy=0 0 1.57079632679
- joint left_thumb_pad_fixed: origin xyz=3.66216494593e-05 -0.028500341515 0.0127727528254 rpy=0 0 0 -> xyz=3.66216494593e-05 -0.028500341515 0.0127727528254 rpy=0.160625387543 1.67750942914e-07 1.35015715552e-08

File: ldjy_retargeting/assets/robots/ldjy_hand/urdf/ldjy_right_hand.urdf (robot description, URDF)
Before this commit: robot ldjy_right_hand, 32 links, 31 joints
Joints:
- joint right_finger1_pad_fixed: origin xyz=-0.000887896997077 -0.00739003330634 0.0202260113406 rpy=0 0 0 -> xyz=-0.000887896997077 -0.00739003330634 0.0202260113406 rpy=1.24252620701 -7.13747250192e-08 -5.10912838703e-08
- joint right_finger2_pad_fixed: origin xyz=-0.000345141712275 -0.00717387617459 0.0207279644612 rpy=0 0 0 -> xyz=-0.000345141712275 -0.00717387617459 0.0207279644612 rpy=1.24005577254 1.45069127377e-07 1.03572263876e-07
- joint right_finger3_pad_fixed: origin xyz=-0.000646578946653 -0.00638898613424 0.0207611224125 rpy=0 0 0 -> xyz=-0.000646578946653 -0.00638898613424 0.0207611224125 rpy=1.19772648334 1.19549859345e-07 8.15891079142e-08
- joint right_finger4_pad_fixed: origin xyz=0.000717825545034 -0.00652127833713 0.030480346822 rpy=0 0 0 -> xyz=0.000717825545034 -0.00652127833713 0.030480346822 rpy=1.19832174357 9.54065941805e-08 6.51537008789e-08
- joint right_retarget_wrist_fixed: origin xyz=-0.015 -0 0.03 rpy=0 0 1.57079632679 -> xyz=-0.0145034869034 0.0111925861623 0.0251133508706 rpy=0 0 1.57079632679
- joint right_thumb_pad_fixed: origin xyz=-3.66216494593e-05 -0.028500341515 0.0127727528254 rpy=0 0 0 -> xyz=-3.66216494593e-05 -0.028500341515 0.0127727528254 rpy=0.160625387543 -1.67750942914e-07 -1.35015715552e-08

File: ldjy_retargeting/assets/robots/openarm_hand/urdf/openarm_bimanual_mano.urdf (robot description, URDF)
Before this commit: robot openarm_bimanual_mano, 82 links, 81 joints
Joints:
- joint left_adapter_to_retarget_wrist: origin xyz=0.0108960117161 -0.0145499234675 -0.0401069474649 rpy=3.14154687609 -0.104536363481 -1.5707794965 -> xyz=-0.000296797861378 -0.0145661583802 -0.0450182202285 rpy=3.14154687609 -0.104536363481 -1.5707794965
- joint left_finger1_pad_frame_fixed: origin xyz=0.000649999999962 0.00450561490399 0.0203260926594 rpy=3.9944714203e-12 1.54044485282 1.57079632679 -> xyz=0.000887896996947 -0.00739003330614 0.0202260113406 rpy=1.24252620701 7.13747254633e-08 5.10864567316e-08
- joint left_finger1_tip_fixed: origin xyz=-4.66040959013e-14 0.00339976361966 0.0297165365339 rpy=0 0 0 -> xyz=-6.07202094561e-14 0.00339976361966 0.0297165365339 rpy=0 0 0
- joint left_finger2_pad_frame_fixed: origin xyz=0.000649999999966 0.00455588780148 0.0203148834496 rpy=4.74242867199e-12 1.54291887718 1.57079632679 -> xyz=0.00034514171214 -0.0071738761746 0.0207279644612 rpy=1.24005577254 -1.45069127377e-07 -1.03577158628e-07
- joint left_finger2_tip_fixed: origin xyz=-4.21546260539e-14 0.00357323373204 0.0297108214506 rpy=0 0 0 -> xyz=-6.10966134148e-14 0.00357323373204 0.0297108214506 rpy=0 0 0
- joint left_finger3_pad_frame_fixed: origin xyz=0.000650000000969 0.00541135856597 0.0201039253082 rpy=3.14159265019 1.55634981875 -1.5707963302 -> xyz=0.000646578946534 -0.00638898613444 0.0207611224125 rpy=1.19772648334 -1.19549859789e-07 -8.15939332766e-08
- joint left_finger3_tip_fixed: origin xyz=1.44288901641e-12 0.00682692933044 0.029504138434 rpy=0 0 0 -> xyz=1.42090123256e-12 0.00682692933044 0.029504138434 rpy=0 0 0
- joint left_finger4_pad_frame_fixed: origin xyz=-0.000527520904384 0.00552645560178 0.0306411188614 rpy=0.127174305263 1.52430090344 1.67999008311 -> xyz=-0.000717825545161 -0.00652127833753 0.030480346822 rpy=1.19832174357 -9.54066303738e-08 -6.5158156759e-08
- joint left_finger4_tip_fixed: origin xyz=0.000305268631434 0.00384935353989 0.0401239267378 rpy=0 0 0 -> xyz=0.000305268631408 0.00384935353989 0.0401239267378 rpy=0 0 0
- joint left_retarget_wrist_fixed: origin xyz=-0.015 -0 0.03 rpy=0 0 1.57079632679 -> xyz=-0.0145034869034 -0.0111925861623 0.0251133508706 rpy=0 0 1.57079632679
- joint left_thumb_pad_frame_fixed: origin xyz=0.000569999999648 -0.0300543833141 0.0124619777338 rpy=3.94084764821e-12 0.0802506835854 1.57079632679 -> xyz=3.66216491132e-05 -0.0285003415151 0.0127727528253 rpy=0.160625387543 1.67754871105e-07 1.34986503225e-08
- joint left_thumb_tip_fixed: origin xyz=-4.16695657022e-13 -0.0399322083727 0.00321148415102 rpy=0 0 0 -> xyz=-4.17114557363e-13 -0.0399322083727 0.00321148415102 rpy=0 0 0
- joint right_adapter_to_retarget_wrist: origin xyz=0.0108960116848 0.0145499234675 -0.0401069474649 rpy=-3.14154687609 -0.104536363481 1.57077949916 -> xyz=-0.000296797892778 0.0145661583504 -0.0450182202285 rpy=-3.14154687609 -0.104536363481 1.57077949916
- joint right_finger1_pad_frame_fixed: origin xyz=-0.00065000000008 0.00450561490359 0.0203260926594 rpy=4.00890431962e-12 -1.54044485282 -1.57079632679 -> xyz=-0.000887896997179 -0.00739003330654 0.0202260113406 rpy=1.24252620701 -7.13747247971e-08 -5.109611112e-08
- joint right_finger1_tip_fixed: origin xyz=-8.1072751647e-14 0.00339976361924 0.0297165365339 rpy=0 0 0 -> xyz=-6.69543208661e-14 0.00339976361924 0.0297165365339 rpy=0 0 0
- joint right_finger2_pad_frame_fixed: origin xyz=-0.000650000000082 0.00455588780152 0.0203148834496 rpy=4.76330086485e-12 -1.54291887718 -1.57079632679 -> xyz=-0.000345141712372 -0.00717387617458 0.0207279644612 rpy=1.24005577254 1.45069127377e-07 1.03567369125e-07
- joint right_finger2_tip_fixed: origin xyz=-8.40410678071e-14 0.00357323373206 0.0297108214506 rpy=0 0 0 -> xyz=-6.50959085599e-14 0.00357323373206 0.0297108214506 rpy=0 0 0
- joint right_finger3_pad_frame_fixed: origin xyz=-0.000650000001049 0.00541135856637 0.0201039253082 rpy=3.14159265019 -1.55634981875 1.5707963302 -> xyz=-0.000646578946728 -0.00638898613404 0.0207611224125 rpy=1.19772648334 1.19549859567e-07 8.15842824409e-08
- joint right_finger3_tip_fixed: origin xyz=-1.50935104949e-12 0.00682692933086 0.029504138434 rpy=0 0 0 -> xyz=-1.48734938783e-12 0.00682692933086 0.029504138434 rpy=0 0 0
- joint right_finger4_pad_frame_fixed: origin xyz=0.00052752090429 0.00552645560258 0.0306411188614 rpy=0.127174305275 -1.52430090344 -1.67999008313 -> xyz=0.000717825544959 -0.00652127833673 0.0304803468221 rpy=1.19832174357 9.54065577652e-08 6.51492454429e-08
- joint right_finger4_tip_fixed: origin xyz=-0.000305268631544 0.00384935354073 0.0401239267378 rpy=0 0 0 -> xyz=-0.000305268631518 0.00384935354073 0.0401239267378 rpy=0 0 0
- joint right_retarget_wrist_fixed: origin xyz=-0.015 -0 0.03 rpy=0 0 1.57079632679 -> xyz=-0.0145034869034 0.0111925861623 0.0251133508706 rpy=0 0 1.57079632679
- joint right_thumb_pad_frame_fixed: origin xyz=-0.000570000000351 -0.0300543833139 0.012461977734 rpy=-3.94118071512e-12 -0.0802506835856 -1.57079632679 -> xyz=-3.66216498046e-05 -0.028500341515 0.0127727528255 rpy=0.160625387543 -1.67747014501e-07 -1.35044921079e-08
- joint right_thumb_tip_fixed: origin xyz=-4.16686502887e-13 -0.0399322083725 0.0032114841512 rpy=0 0 0 -> xyz=-4.16295748377e-13 -0.0399322083726 0.0032114841512 rpy=0 0 0
